Commit message: Add TurtleBot3 Waffle Pi URDF and related configurations
- Introduced URDF and XACRO files for the TurtleBot3 Waffle Pi model.
- Updated launch files to support the new robot model, including spawn and navigation configurations.
- Added costmap and DWA local planner parameters specific to the Waffle Pi.
- Modified existing launch files to accommodate the new robot model while maintaining compatibility with the TurtleBot3 Burger.
- Ensured that all necessary dependencies are included in package.xml files.

File: src/mr_description/urdf/project/turtlebot3_waffle_pi.gazebo.xacro (robot description, xacro)
@@ -1,6 +1,6 @@
 <?xml version="1.0"?>
-<robot name="turtlebot3_burger_sim" xmlns:xacro="http://ros.org/wiki/xacro">
+<robot name="turtlebot3_waffle_pi_gazebo" xmlns:xacro="http://ros.org/wiki/xacro">
   <xacro:arg name="laser_visual" default="false"/>
-  <xacro:arg name="imu_visual"   default="false"/>
+  <xacro:arg name="imu_visual" default="false"/>
   <xacro:arg name="wheel_mu" default="1.0"/>
   <gazebo reference="base_link">
@@ -27,5 +27,14 @@
     <material>Gazebo/FlatBlack</material>
   </gazebo>
-  <gazebo reference="caster_back_link">
+  <gazebo reference="caster_back_right_link">
+    <mu1>0.1</mu1>
+    <mu2>0.1</mu2>
+    <kp>1000000.0</kp>
+    <kd>100.0</kd>
+    <minDepth>0.001</minDepth>
+    <maxVel>1.0</maxVel>
+    <material>Gazebo/FlatBlack</material>
+  </gazebo>
+  <gazebo reference="caster_back_left_link">
     <mu1>0.1</mu1>
     <mu2>0.1</mu2>
@@ -44,5 +53,5 @@
   </gazebo>
   <gazebo>
-    <plugin name="turtlebot3_burger_controller" filename="libgazebo_ros_diff_drive.so">
+    <plugin name="turtlebot3_waffle_pi_controller" filename="libgazebo_ros_diff_drive.so">
       <commandTopic>cmd_vel</commandTopic>
       <odometryTopic>odom</odometryTopic>
@@ -58,8 +67,8 @@
       <leftJoint>wheel_left_joint</leftJoint>
       <rightJoint>wheel_right_joint</rightJoint>
-      <wheelSeparation>0.160</wheelSeparation>
+      <wheelSeparation>0.287</wheelSeparation>
       <wheelDiameter>0.066</wheelDiameter>
       <wheelAcceleration>1</wheelAcceleration>
-      <wheelTorque>10</wheelTorque>
+      <wheelTorque>20</wheelTorque>
       <rosDebugLevel>na</rosDebugLevel>
     </plugin>
@@ -74,21 +83,4 @@
       <gaussianNoise>0.0</gaussianNoise>
       <updateRate>0</updateRate>
-      <imu>
-        <noise>
-          <type>gaussian</type>
-          <rate>
-            <mean>0.0</mean>
-            <stddev>2e-4</stddev>
-            <bias_mean>0.0000075</bias_mean>
-            <bias_stddev>0.0000008</bias_stddev>
-          </rate>
-          <accel>
-            <mean>0.0</mean>
-            <stddev>1.7e-2</stddev>
-            <bias_mean>0.1</bias_mean>
-            <bias_stddev>0.001</bias_stddev>
-          </accel>
-        </noise>
-      </imu>
     </plugin>
   </gazebo>

File: src/mr_description/urdf/turtlebot3_waffle_pi.urdf (robot description, URDF)
Before this commit: robot turtlebot3_burger, 7 links, 6 joints
Links:
- removed link ${namespace}caster_back_link
- added link ${namespace}camera_link; collision box size=0.015 0.030 0.027
- added link ${namespace}camera_rgb_frame
- added link ${namespace}camera_rgb_optical_frame
- added link ${namespace}caster_back_left_link, mass 0.005; collision box size=0.030 0.009 0.020
- added link ${namespace}caster_back_right_link, mass 0.005; collision box size=0.030 0.009 0.020
- link ${namespace}base_link: mass 8.2573504e-01 -> 1.3729096e+00; geometry collision box size=0.266 0.266 0.094; visual mesh filename=package://mr_description/meshes/bases/waffle_pi_base.stl scale=0.001 0.001 0.001
Joints:
- removed joint ${namespace}caster_back_joint
- added joint ${namespace}camera_joint: type fixed, parent ${namespace}base_link, child ${namespace}camera_link, origin xyz=0.073 -0.011 0.084 rpy=0 0 0
- added joint ${namespace}camera_rgb_joint: type fixed, parent ${namespace}camera_link, child ${namespace}camera_rgb_frame, origin xyz=0.003 0.011 0.009 rpy=0 0 0
- added joint ${namespace}camera_rgb_optical_joint: type fixed, parent ${namespace}camera_rgb_frame, child ${namespace}camera_rgb_optical_frame, origin xyz=0 0 0 rpy=-1.57 0 -1.57
- added joint ${namespace}caster_back_left_joint: type fixed, parent ${namespace}base_link, child ${namespace}caster_back_left_link, origin xyz=-0.177 0.064 -0.004 rpy=-1.57 0 0
- added joint ${namespace}caster_back_right_joint: type fixed, parent ${namespace}base_link, child ${namespace}caster_back_right_link, origin xyz=-0.177 -0.064 -0.004 rpy=-1.57 0 0
- joint ${namespace}base_joint: origin xyz=0.0 0.0 0.010 rpy=0 0 0 -> xyz=0 0 0.010 rpy=0 0 0
- joint ${namespace}imu_joint: origin xyz=-0.032 0 0.068 rpy=0 0 0 -> xyz=0.0 0 0.068 rpy=0 0 0
- joint ${namespace}scan_joint: origin xyz=-0.032 0 0.172 rpy=0 0 0 -> xyz=-0.064 0 0.122 rpy=0 0 0
- joint ${namespace}wheel_left_joint: origin xyz=0.0 0.08 0.023 rpy=-1.57 0 0 -> xyz=0.0 0.144 0.023 rpy=-1.57 0 0
- joint ${namespace}wheel_right_joint: origin xyz=0.0 -0.080 0.023 rpy=-1.57 0 0 -> xyz=0.0 -0.144 0.023 rpy=-1.57 0 0
