Commit message: feat: Add WPB Home Mani model and navigation configurations with simulation enhancements

File: src/mr_description/urdf/wpb_home/simulation/wpb_home_mani_model.urdf.xacro (robot description, xacro)
@@ -161,4 +161,9 @@
       <origin rpy="0 0 0" xyz="0 0 0"/>
     </visual>
+    <inertial>
+      <origin xyz="0 0 0" rpy="0 0 0"/>
+      <mass value="0.01"/>
+      <inertia ixx="0.000001" ixy="0.0" ixz="0.0" iyy="0.000001" iyz="0.0" izz="0.000001"/>
+    </inertial>
   </link>
   <joint name="laser_joint" type="fixed">

File: src/mr_description/urdf/wpb_home/simulation/wpb_home_sim.urdf.xacro (robot description, xacro)
@@ -1,5 +1,5 @@
 <?xml version="1.0"?>
 <robot name="wpb_home_simulation" xmlns:xacro="http://ros.org/wiki/xacro">
-  <xacro:include filename="$(find mr_description)/urdf/wpb_home/wpb_home.urdf"/>
+  <xacro:include filename="$(find mr_description)/urdf/wpb_home/simulation/wpb_home_model.urdf.xacro"/>
   <xacro:include filename="$(find mr_description)/urdf/wpb_home/simulation/wpb_home_gazebo_plugins.xacro"/>
   <xacro:wpb_home_simulation_plugins include_mani_joints="false"/>
